File: GuavaPi/GuavaPi.kicad_sch (KiCad schematic)
At the start: 1 part

Commit message: Updated Schematic Sheets
Parts:
- removed U1: ~, symbol Allwinner_H616:Allwinner_H616
Other:
- added sheet GPIO (GuavaPi_GPIO.kicad_sch)
- added sheet Peripherals (GuavaPi_Peripherals.kicad_sch)
- added sheet Power (GuavaPi_Power.kicad_sch)
- added sheet SDRAM (GuavaPi_SDRAM.kicad_sch)
